File: assets/KiCAD/Template/Template.kicad_sch (KiCad schematic)
At the start: 19 parts, among them U1 ADC0820CCN, U10 74LS151, U11 CH552G, U2 74HC595, U3 74HC164, U4 74HC165, U5 74HC4051, U6 74LS49, U7 74LS148, U8 74LS145, U9 74LS147

Commit message: Added bloom!
Parts:
- removed C3: 10uF, Capacitor_THT:CP_Radial_D5.0mm_P2.00mm, symbol Device:C_Polarized_US
- removed U10: 74LS151, symbol 74xx:74LS151
- removed U11: CH552G, Package_SO:SOP-16_3.9x9.9mm_P1.27mm, symbol EasyEDA:CH552G
- removed U2: 74HC595, symbol 74xx:74HC595
- removed U3: 74HC164, symbol 74xx:74HC164
- removed U4: 74HC165, symbol 74xx:74HC165
- removed U5: 74HC4051, symbol 74xx:74HC4051
- removed U6: 74LS49, Package_DIP:DIP-14_W7.62mm_Socket_LongPads, symbol 74xx:74LS49
- removed U7: 74LS148, symbol 74xx:74LS148
- removed U8: 74LS145, symbol 74xx:74LS145
- removed U9: 74LS147, symbol 74xx:74LS147
- added C3, C4: 100nF, Capacitor_THT:C_Disc_D5.0mm_W2.5mm_P2.50mm, symbol Device:C
- added LED1: SM410561N, EasyEDA:LED-SEG-TH_10P-L12.7-W19.0-P2.54-S15.24-BL, symbol EasyEDA:SM410561N
- added R2, R3, R4, R5, R6, R7: 470, Resistor_THT:R_Axial_DIN0207_L6.3mm_D2.5mm_P10.16mm_Horizontal, symbol Device:R_US
- added U2: 74LS47, Package_DIP:DIP-16_W7.62mm_Socket_LongPads, symbol 74xx:74LS47
- added U3: 74LS283, Package_DIP:DIP-16_W7.62mm_Socket_LongPads, symbol 74xx:74LS283
- added U6: 74HC165, Package_DIP:DIP-16_W7.62mm_Socket_LongPads, symbol 74xx:74HC165
- added U7: 74HC595, Package_DIP:DIP-16_W7.62mm_Socket_LongPads, symbol 74xx:74HC595
- C2: value 100nF -> 1nF
- R1: value 1K -> 470
Connections:
- net +5V: now also C1.1, U1.12 (VREF+), U1.20 (VCC), C3.1, LED1.3 (G1), LED1.5 (dp), LED1.8 (G1), U2.16 (VCC), U2.3 (LT), U2.4 (BI), U2.5 (RBI), U3.16 (VCC), U3.7 (C0), U6.16 (VCC), U7.16 (VCC)
- net GND: now also C1.2, C2.2, U1.10 (GND), U1.11 (VREF-), U1.13 (~{CS}), U1.7 (MODE), C3.2, C4.2, U2.8 (GND), U3.11 (B4), U3.15 (B3), U3.2 (B2), U3.6 (B1), U3.8 (GND), U6.8 (GND), U7.13 (~{OE}), U7.8 (GND)
- net at C2.1: now also U1.8 (~{RD}), U1.9 (~{INT}); no longer C1.1
- net ANALOG: now reaches U1.1 (VIN)
- net ANALOG: now also C4.1
- net D4: now reaches U1.14 (DB4)
- net D4: now also U6.3 (D4), U7.4 (QE)
- net D5: now reaches U1.15 (DB5)
- net D5: now also U6.4 (D5), U7.5 (QF)
- net D6: now reaches U1.16 (DB6)
- net D6: now also U6.5 (D6), U7.6 (QG)
- net D7: now reaches U1.17 (DB7)
- net D7: now also U6.6 (D7), U7.7 (QH)
- net D0: now reaches U1.2 (DB0)
- net D0: now also U6.11 (D0), U7.15 (QA)
- net D1: now reaches U1.3 (DB1)
- net D1: now also U6.12 (D1), U7.1 (QB)
- net D2: now reaches U1.4 (DB2)
- net D2: now also U6.13 (D2), U7.2 (QC)
- net D3: now reaches U1.5 (DB3)
- net D3: now also U6.14 (D3), U7.3 (QD)
- net a: now reaches R1.1
- net a: now also LED1.7 (a)
- net at R1.2: now also U2.13 (a)
- new net: R5.2, U2.9 (e)
- new net: R4.2, U2.10 (d)
- new net: R3.2, U2.11 (c)
- new net: R2.2, U2.12 (b)
- new net: R7.2, U2.14 (g)
- new net: R6.2, U2.15 (f)
- new net ID_IN_0: U2.7 (A), U3.5 (A1)
- new net ID_IN_1: U2.1 (B), U3.3 (A2)
- new net ID_IN_2: U2.2 (C), U3.14 (A3)
- new net ID_IN_3: U2.6 (D), U3.12 (A4)
- new net ID_OUT_0: U3.4 (S1)
- new net ID_OUT_1: U3.1 (S2)
- new net ID_OUT_2: U3.13 (S3)
- new net ID_OUT_3: U3.10 (S4)
- new net PCLK: U6.2 (CP)
- new net PCLR: U6.15 (~{CE})
- new net PDATA_IN: U6.10 (DS)
- new net PDATA_OUT: U6.9 (Q7)
- new net PLATCH: U6.1 (~{PL})
- new net SCLK: U7.11 (SRCLK)
- new net SCLR: U7.10 (~{SRCLR})
- new net SDATA_IN: U7.14 (SER)
- new net SLATCH: U7.12 (RCLK)
- new net b: LED1.6 (b), R2.1
- new net c: LED1.4 (c), R3.1
- new net d: LED1.2 (d), R4.1
- new net e: LED1.1 (e), R5.1
- new net f: LED1.9 (f), R6.1
- new net g: LED1.10 (g), R7.1
- no-connect marks 0 -> 6
Other:
- note added: "Identity"
- moved on the sheet: H1, H2, H3, H4, U1

Commit message: added terrain to opencl
Parts:
- added C5, C7: 100nF, Capacitor_THT:C_Disc_D5.0mm_W2.5mm_P2.50mm, symbol Device:C
- added C6: 10uF, Capacitor_THT:CP_Radial_D5.0mm_P2.00mm, symbol Device:C_Polarized_US
- added R10, R11: 10K, Resistor_THT:R_Axial_DIN0207_L6.3mm_D2.5mm_P10.16mm_Horizontal, symbol Device:R_US
- added R8, R9: 5.1K, Resistor_THT:R_Axial_DIN0207_L6.3mm_D2.5mm_P10.16mm_Horizontal, symbol Device:R_US
- added SW1: BOOT, Button_Switch_THT:SW_PUSH_6mm, symbol Switch:SW_Push
- added SW2: RESET, Button_Switch_THT:SW_PUSH_6mm, symbol Switch:SW_Push
- added U4: CH552G, Package_SO:SOP-16_3.9x9.9mm_P1.27mm, symbol EasyEDA:CH552G
- added USB1: TYPEC, EasyEDA:USB-C-SMD_TYPEC-302-BRP16SC16, symbol EasyEDA:TYPEC-302-BRP16SC16
- U2, U3, U6, U7: footprint Package_DIP:DIP-16_W7.62mm_Socket_LongPads -> Package_SO:SOP-16_3.9x9.9mm_P1.27mm
Connections:
- net +5V: now also C5.1, C6.1, U4.15 (VCC/VDD), USB1.11 (VBUS), USB1.2 (VBUS)
- net GND: now also C5.2, C6.2, C7.1, R11.2, R8.2, R9.2, U4.14 (GND/VSS), USB1.1 (GND), USB1.12 (GND), USB1.13 (SHELL), USB1.14 (SHELL), USB1.15 (SHELL), USB1.16 (SHELL)
- new net: R11.1, SW2.1, U4.6 (RST/T2EX_/CAP2_)
- new net: C7.2, SW1.1, SW2.2, U4.16 (V33)
- new net: R10.2, SW1.2
- new net: R9.1, USB1.10 (CC2)
- new net: R8.1, USB1.4 (CC1)
- new net D+: R10.1, U4.12 (P3.6/UDP), USB1.6 (DP1), USB1.8 (DP2)
- new net D-: U4.13 (P3.7/UDM), USB1.5 (DN2), USB1.7 (DN1)
- no-connect marks 6 -> 8
Other:
- note removed: "Identity"
- moved on the sheet: C1, C2, C3, C4, H1, H2, H3, H4, U1, U6, U7
